File: KiCAD/Garage133.kicad_sch (KiCad schematic)
At the start: 24 parts, among them U3 SHTC3

Commit message: Version 2.1.0: four sonars, USB-C (#26)
## [2.1.0] - 2026-10-14

### Added
- **Hardware Board v3.1 & Enclosure Updates**: KiCAD PCB updates for
board v3.1 with revised BOM, updated 3D printable enclosure (better
SHTC3 thermal isolation, labeled connectors, improved USB-C port
clearance), and solder stencil support frame model.
- **HMM Visualization & Retraining Workflow**: Added
`analysis/hmm_to_svg.py` to generate SVG state transition diagrams from
trained HMM models, and added characterization workflow in
`analysis/retrain.py`.

### Changed
- **Sonar Watchdog & Timeout Stability**: Added sonar ping timeout
handling to prevent blocking pulses from triggering the ESP32 hardware
watchdog.

### Removed
- **Retired Legacy Hardware**: Removed firmware and PlatformIO
configuration support for legacy Classic ESP32 boards (Board v1/v2 /
`node32s`), focusing entirely on Board v3.x (ESP32-S3).

## [2.0.0] - 2026-08-21

### Added
- **Hardware Board v3.0 & ESP32-S3 Support**: Added PlatformIO
configuration (`usb_s3`), pin assignments for ESP32-S3, updated
schematic/PCB designs, and refreshed solder stencil fixture 3D models.
- **Quad-Sonar Support**: Integrated dual ultrasonic sensors per side (4
total) with updated state classification logic, training pipeline, and
retrained HMM models.
- **Home Assistant Probability Export**: Exported garage state
probabilities (`probOpen`, `probCar`, `probEmpty`) via Home Assistant
MQTT discovery.

### Changed
- **Svelte Build Tooling**: Pinned `svelteesp32` to v3.2.5 and updated
CI workflows to Node 22 for reproducible builds.
- **Dependency & Workflow Upgrades**: Upgraded `og3` to v0.6.3,
`og3x-oled` to v0.6.1, and updated GitHub Actions workflows to latest
versions.
Parts:
- added D_R3: YLW, LED_SMD:LED_0603_1608Metric, symbol Device:LED
- added Rl5: 1k, Resistor_SMD:R_0603_1608Metric, symbol Device:R
Connections:
- net GND: now also Rl5.1
- new net: D_R3.1 (K), Rl5.2
- new net LED1: D_R3.2 (A)
